File: gate_driver.kicad_sch (KiCad schematic)
At the start: 9 parts, among them U5 DRV8353SRTAR

Commit message: Add STM32G474METx MCU sheet wired to the pin plan
MCU sheet follows Comms Component Selection.ioc. Gate driver switched to
6-PWM (INLA/B/C split from MOTOR_HIZ) to match TIM1 CHx/CHxN. Root nets
renamed to the pin-plan names (PWM_xH/xL, GATE_EN, DRV_*, CURR_A/B/C).

Co-Authored-By: Claude Opus 5.5 <noreply@anthropic.com>
Connections:
- removed net MOTOR_HIZ: U5.33 (INLA), U5.35 (INLB), U5.37 (INLC)
- new net INLA: U5.33 (INLA)
- new net INLB: U5.35 (INLB)
- new net INLC: U5.37 (INLC)
Changed lines of the file:
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@@
 		(rev "A")
 		(comment 1 "Derived from mjbots moteus-x1 r1 (Apache-2.0), https://github.com/mjbots/moteus")
+		(comment 2 "Modified: INLA/INLB/INLC split out (was MOTOR_HIZ) for 6-PWM mode")
 	)
 	(junction
@@
 		)
 	)
-	(hierarchical_label "MOTOR_HIZ"
+	(hierarchical_label "INLB"
 		(shape input)
 		(at 73.66 85.09 180)
@@
 		)
 	)
-	(hierarchical_label "MOTOR_HIZ"
+	(hierarchical_label "INLC"
 		(shape input)
 		(at 73.66 92.71 180)
@@
 		)
 	)
-	(hierarchical_label "MOTOR_HIZ"
+	(hierarchical_label "INLA"
 		(shape input)
 		(at 73.66 77.47 180)
