File: stm32g474.kicad_sch (KiCad schematic)
At the start: 1 part, among them U1 STM32G474METx

Commit message: MCU sheet edits: move VBUS to PA2, add USART3 on PE15/PB10
Schematic files re-saved in KiCad 10 format. Ignore VS Code .history/.

Co-Authored-By: Claude Opus 5.5 <noreply@anthropic.com>
Connections:
- net +3V: no longer U1.16 (VDD), U1.28 (VREF+), U1.29 (VDDA), U1.41 (VDD), U1.51 (VDD), U1.62 (VDD), U1.80 (VDD)
- net GND: no longer U1.15 (VSS), U1.40 (VSS), U1.50 (VSS), U1.61 (VSS), U1.79 (VSS)
- net VBUS: now also U1.14 (PA2); no longer U1.38 (PE15)
- net USART3_TX: now reaches U1.39 (PB10)
- new net: U1.15 (VSS), U1.40 (VSS), U1.50 (VSS), U1.61 (VSS), U1.79 (VSS)
- new net: U1.16 (VDD), U1.41 (VDD), U1.51 (VDD), U1.62 (VDD), U1.80 (VDD)
- new net USART3_RX: U1.38 (PE15)
- no-connect marks 23 -> 21

Commit message: Fix MCU power wiring and add USART3 sheet pins
Reconnect the +3V rail (shifted off the VBAT/VDDA stubs), add the missing
VREF+ and VSS wires, and add USART3_TX/RX pins to the MCU sheet symbol.

Co-Authored-By: Claude Opus 5.5 <noreply@anthropic.com>
Connections:
- net +3V: now also U1.16 (VDD), U1.28 (VREF+), U1.29 (VDDA), U1.41 (VDD), U1.51 (VDD), U1.62 (VDD), U1.80 (VDD)
- net GND: now also U1.15 (VSS), U1.40 (VSS), U1.50 (VSS), U1.61 (VSS), U1.79 (VSS)
Changed lines of the file:
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@@
 	(wire
 		(pts
-			(xy 196.85 76.2) (xy 212.09 76.2)
+			(xy 195.58 76.2) (xy 210.82 76.2)
 		)
 		(stroke
+			(width 0)
+			(type default)
+		)
+	)
+	(wire
+		(pts
+			(xy 177.8 88.9) (xy 182.88 88.9)
+		)
+		(stroke
+			(width 0)
+			(type default)
+		)
+	)
+	(wire
+		(pts
+			(xy 203.2 195.58) (xy 203.2 200.66)
+		)
+		(stroke
