File: hardware/h_bridge.kicad_sch (KiCad schematic)
At the start: 8 parts, among them Q1 FDMT80080DC, Q2 FDMT80080DC, X1 Conn_01x01

Commit message: Clean up schematic ERC; add project symbol library; update README
Fix dangling labels, floating pins and pin types across the sheets so
ERC reports 0 errors (see hardware/CHANGES.txt). Add PWR_FLAGs and move
TCAN1042GV, MA702GQ and the EMI filter to nexus_drive.kicad_sym.

Update the README layout, specs and schematic review status.

Co-Authored-By: Claude Opus 5.5 <noreply@anthropic.com>
Other:
- moved on the sheet: C24, D4, Q1, Q2, X1
