File: hardware/stm32g474.kicad_sch (KiCad schematic)
At the start: 1 part, among them U1 STM32G474METx

Commit message: Add CAN FD and encoder sheets; update MCU sheet and root schematic
Co-Authored-By: Claude Opus 5.5 <noreply@anthropic.com>
Parts:
- added C? (x2): 12pF, symbol Device:C_Small
- added C? (x2): 4.7uF, symbol Device:C_Small
- added C? (x8): 100nF, symbol Device:C_Small
- added C?: 1uF, symbol Device:C_Small
- added FB?: 600 Ohm @ 100MHz (0603), symbol Device:FerriteBead_Small
- added J?: Conn_01x05_Pin, Connector_PinHeader_1.27mm:PinHeader_1x05_P1.27mm_Vertical, symbol Connector:Conn_01x05_Pin
- added JP?: SolderJumper_2_Open, symbol Jumper:SolderJumper_2_Open
- added R?: 10k, symbol Device:R_Small
- added Y1: 16MHz, symbol Device:Crystal_Small
Connections:
- net +3V: now also C?.1, C?.1, C?.1, C?.1, C?.1, C?.1, C?.1, C?.1, FB?.1, J?.1 (Pin_1), JP?.1 (A); no longer U1.28 (VREF+), U1.29 (VDDA)
- net BOOT0: now also JP?.2 (B), R?.1
- net GND: now also C?.2, C?.2, C?.2, C?.2, C?.2, C?.2, C?.2, C?.2, C?.2, C?.2, C?.2, C?.2, C?.2, J?.5 (Pin_5), R?.2
- net NRST: now also C?.1, J?.4 (Pin_4)
- net OSC_IN: now also C?.1, Y1.1
- net OSC_OUT: now also C?.1, Y1.2
- net SWCLK: now also J?.3 (Pin_3)
- net SWDIO: now also J?.2 (Pin_2)
- new net +3VA: C?.1, C?.1, FB?.2, U1.28 (VREF+), U1.29 (VDDA)
Other:
- note added: "D1: VBAT / VDD decoupling. 100nF x6 (VBAT pin 1, VDD pins 16/41/51/62/80) + 4.7uF x2 bulk."
- note added: "D2: +3VA = +3V via ferrite bead, feeds VDDA (pin 29) and VREF+ (pin 28)."
- note added: "D3-D5: NRST cap, SWD header, BOOT0 pulldown + solder jumper to +3V."
- note added: "D6: 16MHz HSE crystal, 2x 12pF C0G load caps."

Commit message: Add sensing sheet; update MCU, CAN FD, encoder and root schematics
Co-Authored-By: Claude Opus 5.5 <noreply@anthropic.com>
Parts:
- added J1: Conn_01x03, symbol Connector_Generic:Conn_01x03
Connections:
- net GND: now also J1.3 (Pin_3)
- net USART3_RX: now also J1.2 (Pin_2)
- net USART3_TX: now also J1.1 (Pin_1)
- net VPH_C: now also U1.10 (PC2); no longer U1.30 (PE7)
- no-connect marks 21 -> 22
Changed lines of the file:
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@@
+	)
+	(no_connect
+		(at 182.88 106.68)
 	)
 	(no_connect
@@
 	(wire
 		(pts
+			(xy 294.64 147.32) (xy 294.64 152.4)
+		)
+		(stroke
+			(width 0)
+			(type default)
+		)
+	)
+	(wire
+		(pts
 			(xy 177.8 175.26) (xy 182.88 175.26)
 		)
@@
 	(wire
 		(pts
+			(xy 294.64 142.24) (xy 299.72 142.24)
+		)
+		(stroke
+			(width 0)
+			(type default)
+		)
+	)
+	(wire
+		(pts
 			(xy 106.68 165.1) (xy 106.68 167.64)
 		)
@@
 	(wire
 		(pts
+			(xy 294.64 147.32) (xy 299.72 147.32)
+		)
+		(stroke
+			(width 0)
+			(type default)
+		)
+	)
+	(wire
+		(pts
 			(xy 223.52 106.68) (xy 228.6 106.68)
 		)
@@
 	(wire
 		(pts
-			(xy 177.8 106.68) (xy 182.88 106.68)
+			(xy 177.8 154.94) (xy 182.88 154.94)
+		)
+		(stroke
+			(width 0)
+			(type default)
+		)
+	)
+	(wire
+		(pts
+			(xy 294.64 144.78) (xy 299.72 144.78)
 		)
 		(stroke
@@
 			(font
 				(size 1.27 1.27)
+			)
+			(justify left bottom)
+		)
+	)
+	(label "USART3_TX"
+		(at 294.64 142.24 0)
+		(effects
+			(font
+				(size 0.762 0.762)
+			)
+			(justify left bottom)
+		)
+	)
+	(label "USART3_RX"
+		(at 294.64 144.78 0)
+		(effects
+			(font
+				(size 0.762 0.762)
 			)
 			(justify left bottom)
@@
 	(hierarchical_label "VPH_C"
 		(shape bidirectional)
-		(at 177.8 106.68 180)
+		(at 177.8 154.94 180)
 		(effects
 			(font
@@
 					(unit 1)
 				)
+			)
+		)
+	)
+	(symbol
+		(lib_id "Connector_Generic:Conn_01x03")
+		(at 304.8 144.78 0)
+		(unit 1)
+		(body_style 1)
+		(exclude_from_sim no)
+		(in_bom yes)
+		(on_board yes)
+		(in_pos_files yes)
+		(dnp no)
+		(fields_autoplaced yes)
+		(property "Reference" "J1"
+			(at 307.34 143.5099 0)
+			(show_name no)
+			(do_not_autoplace no)
+			(effects
+				(font
+					(size 1.27 1.27)
+				)
+				(justify left)
+			)
+		)
+		(property "Value" "Conn_01x03"
+			(at 307.34 146.0499 0)
+			(show_name no)
+			(do_not_autoplace no)
+			(effects
+				(font
+					(size 1.27 1.27)
+				)
+				(justify left)
+			)
+		)
+		(property "Footprint" ""
+			(at 304.8 144.78 0)
+			(hide yes)
+			(show_name no)
+			(do_not_autoplace no)
+			(effects
+				(font
+					(size 1.27 1.27)
+				)
+			)
+		)
+		(property "Datasheet" ""
+			(at 304.8 144.78 0)
+			(hide yes)
+			(show_name no)
+			(do_not_autoplace no)
+			(effects
+				(font
+					(size 1.27 1.27)
+				)
+			)
+		)
+		(property "Description" "Generic connector, single row, 01x03, script generated (kicad-library-utils/schlib/autogen/connector/)"
+			(at 304.8 144.78 0)
+			(hide yes)
+			(show_name no)
+			(do_not_autoplace no)
+			(effects
+				(font
+					(size 1.27 1.27)
+				)
+			)
+		)
+		(pin "1"
+		)
+		(pin "2"
+		)
+		(pin "3"
+		)
+		(instances
+			(project "nexus_drive"
+				(path "/2d97709d-a8ce-4889-9b37-2fa808653238/5f0c7e2a-3b1d-4c8e-9a6f-2d4b8e1c7a90"
+					(reference "J1")
+					(unit 1)
+				)
+			)
+		)
+	)
+	(symbol
+		(lib_id "power:GND")
+		(at 294.64 152.4 0)
+		(unit 1)
+		(body_style 1)
+		(exclude_from_sim no)
+		(in_bom yes)
+		(on_board yes)
+		(in_pos_files yes)
+		(dnp no)
+		(fields_autoplaced yes)
+		(property "Reference" "#PWR01"
+			(at 294.64 158.75 0)
+			(hide yes)
+			(show_name no)
+			(do_not_autoplace no)
+			(effects
+				(font
+					(size 1.27 1.27)
+				)
+			)
+		)
+		(property "Value" "GND"
+			(at 294.64 157.48 0)
+			(show_name no)
+			(do_not_autoplace no)
+			(effects
+				(font
+					(size 1.27 1.27)
+				)
+			)
+		)
+		(property "Footprint" ""
+			(at 294.64 152.4 0)
+			(hide yes)
+			(show_name no)
+			(do_not_autoplace no)
+			(effects
+				(font
+					(size 1.27 1.27)
+				)
+			)
+		)
+		(property "Datasheet" ""
+			(at 294.64 152.4 0)
+			(hide yes)
+			(show_name no)
+			(do_not_autoplace no)
+			(effects
+				(font
+					(size 1.27 1.27)
+				)
+			)
+		)
+		(property "Description" "Power symbol creates a global label with name \"GND\" , ground"
+			(at 294.64 152.4 0)
+			(hide yes)
+			(show_name no)
+			(do_not_autoplace no)
+			(effects
+				(font
+					(size 1.27 1.27)
+				)
+			)
+		)
+		(pin "1"
+		)
+		(instances
+			(project "nexus_drive"
+				(path "/2d97709d-a8ce-4889-9b37-2fa808653238/5f0c7e2a-3b1d-4c8e-9a6f-2d4b8e1c7a90"
+					(reference "#PWR01")
+					(unit 1)
+				)

Commit message: Clean up schematic ERC; add project symbol library; update README
Fix dangling labels, floating pins and pin types across the sheets so
ERC reports 0 errors (see hardware/CHANGES.txt). Add PWR_FLAGs and move
TCAN1042GV, MA702GQ and the EMI filter to nexus_drive.kicad_sym.

Update the README layout, specs and schematic review status.

Co-Authored-By: Claude Opus 5.5 <noreply@anthropic.com>
Parts:
- gave numbers to parts that had none: 17
Connections:
- no-connect marks 22 -> 21
